File: Hardware/bib.brd (EAGLE design)
At the start: 122 x 90 mm, 65 parts, among them IC1 7805TV, IC2 7812TV, IC3 LM1117V33TV, IC4 74HC157D

Commit message: fixed errors bringing this up to V1.1
Parts:
- removed R12: 150, resistor:R0805
- added JP1: AVR-ISP-6VERT, avr-7:AVR-ISP-6
- added R2: 150, resistor:R0805
- added R3: 10k, resistor:R0805
- added U$2, U$5, U$6: (no value), holes:3,0
- U$4: value AVR-ISP-6-EDGE -> (none); device my_lib:6PAD_ISP -> holes:3,0
- moved U$4 7.35 mm to (123.5, 12.0), turned to 0 degrees
- moved SV8 3.29 mm to (119.9, 81.2), turned to 90 degrees
- moved I2C1 2.00 mm to (18.2, 13.0)
- moved I2C2 2.00 mm to (23.1, 13.0)
- moved I2C3 2.00 mm to (28.0, 13.0)
Connections:
- removed net EN2: PCB2.A3, SV4.3
- removed net MISO: U$3.6, U$4.MISO
- removed net N$33: LED4.A, R12.1
- removed net SEL/RST: IC4.1, R12.2, U$3.1, U$4.RST
- new net MEH: PCB2.2, SV6.6
- new net MISO/SEL: IC4.1, JP1.1, R2.2, U$3.6
- new net N$2: LED4.A, R2.1
- new net RST: JP1.5, R3.1, U$3.1
- net +5V: now also JP1.2, R3.2; no longer U$4.VCC
- net GND: now also JP1.6; no longer U$4.GND
- net MOSI: now also JP1.4; no longer U$4.MOSI
- net SCK: now also JP1.3; no longer U$4.SCK
- net TX4: now also PCB2.A3, SV4.3; no longer PCB2.2, SV6.6
Routing:
- net MISO/SEL: track 0.00 -> 105.4 mm, vias 0 -> 4
- net SEL/RST: track 103.6 -> 0.00 mm, vias 2 -> 0
- net MISO: track 40.2 -> 0.00 mm
- net RST: track 0.00 -> 38.2 mm
- net GND: track 59.8 -> 28.7 mm, vias 16 -> 3
- net TX4: track 136.6 -> 110.1 mm
- net EN2: track 5.04 -> 0.00 mm
- net SCK: track 99.9 -> 96.0 mm
- net N$2: track 0.00 -> 2.78 mm
- net N$33: track 2.75 -> 0.00 mm
- net SDA: track 48.5 -> 46.5 mm
- net SCL: track 40.6 -> 38.6 mm
- net MOSI: track 40.3 -> 41.8 mm, vias 1 -> 2
- net +5V: track 44.4 -> 44.1 mm, vias 8 -> 7
Other:
- outline, holes or cut-outs redrawn
- board text added: "Boat Interface Board V1.1"
- board text added: "SERVOS IN"
- board text added: "SERVOS OUT"
- board text removed: "Boat Interface Board V1"
- board text removed: "MISO"
- board text removed: "MOSI"
- board text removed: "RST"
- board text removed: "SCK"
